File: Placa_perro/Placa_perro.kicad_pcb (KiCad board)
At the start: 2 copper layers, 221.6 x 131.2 mm, 51 parts, among them J1 S_TEMPERATURA, J11 PANTALLA, J12 ENTRADA, J13 OPTO, J14 SALIDA_3.3v, J16 12v, J17 5v, J18 3.3v, J19 GND, J2 LDR, J20 LDR, J22 SALIDA_RELE_1, J4 S_GAS1, J5 S_GAS2, J6 USB_B, J7 Placa control, J8 Placa control, K2 Relay_SPDT, Q2 BC337, SW1 SW_DPDT_x2, SW10 SW_Push, SW11 SW_Push, SW12 SW_Push, SW13 SW_Push, SW9 SW_Push, U1 ESP32-Devkit-V1, U2 LM7805_TO220, U3 PC817

Commit message: terminada
Parts:
- removed J7: Placa control, Connector_PinSocket_2.54mm:PinSocket_1x10_P2.54mm_Vertical
- removed J8: Placa control, Connector_PinHeader_2.54mm:PinHeader_1x10_P2.54mm_Vertical
- added J10: Conn_01x06_Pin, Connector_Molex:Molex_KK-254_AE-6410-06A_1x06_P2.54mm_Vertical, F.Cu at (90.3, 106.2)
- added J15: Conn_01x04_Pin, Connector_Molex:Molex_KK-254_AE-6410-04A_1x04_P2.54mm_Vertical, F.Cu at (90.4, 89.9)
- added J21: Conn_01x06_Pin, Connector_Molex:Molex_KK-254_AE-6410-06A_1x06_P2.54mm_Vertical, F.Cu at (114.4, 180.3)
- added J23: Conn_01x04_Pin, Connector_Molex:Molex_KK-254_AE-6410-04A_1x04_P2.54mm_Vertical, F.Cu at (98.0, 180.3)
- added REF**: MountingHole_3.2mm_M3, MountingHole:MountingHole_3.2mm_M3, F.Cu at (85.0, 63.0)
- added REF**: MountingHole_3.2mm_M3, MountingHole:MountingHole_3.2mm_M3, F.Cu at (166.7, 179.5)
- added REF**: MountingHole_3.2mm_M3, MountingHole:MountingHole_3.2mm_M3, F.Cu at (166.0, 127.0)
- added REF**: MountingHole_3.2mm_M3, MountingHole:MountingHole_3.2mm_M3, F.Cu at (85.0, 127.0)
- added REF**: MountingHole_3.2mm_M3, MountingHole:MountingHole_3.2mm_M3, F.Cu at (166.7, 163.5)
- added REF**: MountingHole_3.2mm_M3, MountingHole:MountingHole_3.2mm_M3, F.Cu at (41.2, 163.5)
- added REF**: MountingHole_3.2mm_M3, MountingHole:MountingHole_3.2mm_M3, F.Cu at (41.2, 179.5)
- added REF**: MountingHole_3.2mm_M3, MountingHole:MountingHole_3.2mm_M3, F.Cu at (166.0, 63.0)
- moved R16 120.9 mm to (53.3, 177.5)
- moved R19 120.9 mm to (133.8, 161.6)
- moved SW11 120.9 mm to (102.6, 173.8)
- moved SW13 120.9 mm to (148.2, 173.8)
- moved R13 120.9 mm to (88.4, 161.6)
- moved R15 120.9 mm to (65.6, 177.5)
- moved R18 120.9 mm to (111.1, 161.6)
- moved SW12 120.9 mm to (125.4, 173.8)
- moved D10 120.9 mm to (47.3, 164.2)
- moved D11 120.9 mm to (47.3, 171.7)
- moved D12 120.9 mm to (47.3, 179.1)
- moved R11 120.9 mm to (65.6, 161.6)
- moved R17 120.9 mm to (53.3, 181.1)
- moved R20 120.9 mm to (156.5, 161.6)
- moved SW10 120.9 mm to (79.8, 173.8)
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Connections:
- R16 pad 2: LED_2 -> LED_1
- R17 pad 2: LED_1 -> LED_2
Routing:
- net +3.3V: track 363.4 -> 397.6 mm
- net RELE_1: track 32.9 -> 21.4 mm
- net Net-(J13-Pin_1): track 7.32 -> 16.7 mm
- net Net-(J13-Pin_2): track 7.89 -> 15.5 mm
- net BOTON_4: track 56.8 -> 62.5 mm
- net Net-(D5-A): track 13.1 -> 18.1 mm
- net Net-(Q2-B): track 9.56 -> 13.6 mm
- net LED_3: track 72.1 -> 68.8 mm
- net BOTON_5: track 63.9 -> 67.1 mm
- net GND: track 545.0 -> 541.8 mm
- net BOTON_3: track 43.9 -> 46.2 mm
- net BOTON_1: track 86.6 -> 85.2 mm
- net BOTON_2: track 62.9 -> 61.8 mm
- net LED_2: track 87.2 -> 86.5 mm
- net +12V: track 24.8 -> 24.3 mm
Other:
- board size 221.6 x 131.2 mm -> 135.2 x 128 mm
