File: Placa_perro/Placa_perro.kicad_sch (KiCad schematic)
At the start: 48 parts, among them J1 S_TEMPERATURA, J10 TEST_POINT1, J11 PANTALLA, J12 ENTRADA, J14 SALIDA_3.3v, J15 ADC, J16 12v, J17 5v, J18 3.3v, J19 GND, J2 LDR, J20 LDR, J21 ADC, J22 SALIDA_RELE_1, J4 S_GAS1, J5 S_GAS2, J6 USB_B, J8 SALIDA_3.3v, J9 SALIDA_RELÉ, K2 Relay_SPDT, Q2 BC337, SW10 SW_Push, SW11 SW_Push, SW12 SW_Push, SW13 SW_Push, SW9 SW_Push, U2 LM7805_TO220

Commit message: esq
Parts:
- removed D10, D11, D12: LED, LED_THT:LED_D3.0mm_Clear, symbol Device:LED
- removed J10: TEST_POINT1, symbol Connector:Conn_01x01_Pin
- removed J8: SALIDA_3.3v, symbol Connector:Conn_01x02_Pin
- removed J9: SALIDA_RELÉ, symbol Connector:Conn_01x02_Pin
- removed R11, R13, R18, R19, R20: 10k, Resistor_THT:R_Axial_DIN0207_L6.3mm_D2.5mm_P7.62mm_Horizontal, symbol Device:R
- removed R15, R16, R17: 120, Resistor_THT:R_Axial_DIN0207_L6.3mm_D2.5mm_P7.62mm_Horizontal, symbol Device:R
- removed SW10, SW11, SW12, SW13, SW9: SW_Push, Button_Switch_THT:SW_PUSH_6mm, symbol Switch:SW_Push
- added J8: Placa control, symbol Connector:Conn_01x10_Pin
- added SW1: SW_DPDT_x2, symbol Switch:SW_DPDT_x2
- added U1: ESP32-Devkit-V1, DOIT_ESP32:DOIT_ESP32_Devkit_mirko, symbol esp32-devkit-v1:ESP32-Devkit-V1
Connections:
- net +12V: now also SW1.1 (A); no longer D4.1 (K)
- net +3.3V: now also J8.1 (Pin_1), U1.30 (3v3); no longer J11.3 (Pin_3)
- net +5V: now also J11.3 (Pin_3), U1.1 (Vin)
- net BOTON_1: now also J8.7 (Pin_7), U1.7 (IO26)
- net BOTON_2: now also J8.6 (Pin_6), U1.6 (IO27)
- net BOTON_3: now also J8.5 (Pin_5), U1.5 (IO14)
- net BOTON_4: now also J8.4 (Pin_4), U1.3 (IO13)
- net BOTON_5: now also J8.3 (Pin_3), U1.4 (IO12)
- net GND: now also J8.2 (Pin_2), U1.2 (GND), U1.29 (GND)
- net LDR: now also U1.27 (IO2)
- net LED_1: now also J8.10 (Pin_10), U1.10 (IO32)
- net LED_2: now also J8.9 (Pin_9), U1.9 (IO33)
- net LED_3: now also J8.8 (Pin_8), U1.8 (IO25)
- net RELE_1: now also U1.26 (IO4)
- net SCL: now also U1.20 (IO21)
- net SDA: now also U1.17 (IO22)
- new net: D4.1 (K), SW1.2 (B)
Other:
- added sheet Placa control (placa_control.kicad_sch)
- note added: "SI o SI con disipador"
- note added: "huella esp32 en kikad??? adc? pull ups sda y scl"
- note removed: "voltaje pantalla SALIDA RELE conecotres varios?? huella esp32 en kikad??? 7805 mucho calor?? adc? pull ups sda y scl us vien conectado?? tema salida rele"
- moved on the sheet: C1, C2, D4, D5, J1, J11, J12, J16, J17, J18, J19, J2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

Commit message: rutee pcb falta molex
Parts:
- removed J15: ADC, Connector_Molex:Molex_KK-254_AE-6410-03A_1x03_P2.54mm_Vertical, symbol Connector:Conn_01x03_Pin
- removed J21: ADC, Connector_PinHeader_2.54mm:PinHeader_1x01_P2.54mm_Vertical, symbol Connector:Conn_01x01_Pin
- removed R12, R14: 10k, Resistor_THT:R_Axial_DIN0207_L6.3mm_D2.5mm_P7.62mm_Horizontal, symbol Device:R
- removed R7: LDR03, OptoDevice:R_LDR_10x8.5mm_P7.6mm_Vertical, symbol Sensor_Optical:LDR03
- added J13: OPTO, TerminalBlock:TerminalBlock_MaiXu_MX126-5.0-02P_1x02_P5.00mm, symbol Connector:Conn_01x02_Pin
- added R21, R23: 18k, Resistor_THT:R_Axial_DIN0207_L6.3mm_D2.5mm_P7.62mm_Horizontal, symbol Device:R
- added R22, R24, R25: 10k, Resistor_THT:R_Axial_DIN0207_L6.3mm_D2.5mm_P7.62mm_Horizontal, symbol Device:R
- added U3: PC817, Package_DIP:DIP-4_W7.62mm, symbol Isolator:PC817
- J1, J4, J5: footprint (none) -> Connector_Molex:Molex_KK-254_AE-6410-04A_1x04_P2.54mm_Vertical
- J11: footprint Connector_PinHeader_2.54mm:PinHeader_1x04_P2.54mm_Vertical -> Connector_Molex:Molex_KK-254_AE-6410-04A_1x04_P2.54mm_Vertical
- J2: footprint (none) -> Connector_Molex:Molex_KK-254_AE-6410-02A_1x02_P2.54mm_Vertical
- J6: footprint (none) -> Connector_USB:USB_B_Lumberg_2411_02_Horizontal
- J8: footprint (none) -> Connector_PinHeader_2.54mm:PinHeader_1x10_P2.54mm_Vertical
- SW1: footprint (none) -> Connector_PinHeader_2.54mm:PinHeader_1x02_P2.54mm_Vertical
Connections:
- net +3.3V: now also J2.2 (Pin_2), U3.4; no longer J1.3 (Pin_3), J2.1 (Pin_1)
- net +5V: now also J1.3 (Pin_3)
- net BOTON_1: now also U1.6 (IO27); no longer U1.7 (IO26)
- net BOTON_2: now also U1.7 (IO26); no longer U1.6 (IO27)
- net BOTON_3: now also U1.8 (IO25); no longer U1.5 (IO14)
- net BOTON_4: now also U1.11 (IO35); no longer U1.3 (IO13)
- net BOTON_5: now also U1.14 (IO36); no longer U1.4 (IO12)
- net GAS1_OUTA: now also U1.10 (IO32), R22.2; no longer J4.2 (Pin_2)
- net GAS2_OUTA: now also U1.9 (IO33), R24.2; no longer J5.2 (Pin_2)
- net GND: now also J12.1 (Pin_1), R21.2, R23.2, R25.2; no longer J12.2 (Pin_2)
- net LDR: now also J2.1 (Pin_1), U1.12 (IO34); no longer J2.2 (Pin_2), U1.27 (IO2)
- net LED_1: now also U1.3 (IO13); no longer U1.10 (IO32)
- net LED_2: now also U1.4 (IO12); no longer U1.9 (IO33)
- net LED_3: now also U1.5 (IO14); no longer U1.8 (IO25)
- net NC_1: now also J22.3 (Pin_3); no longer J22.1 (Pin_1)
- net NO_1: now also J22.1 (Pin_1); no longer J22.3 (Pin_3)
- net RELE_1: now also U1.25 (IO16); no longer U1.26 (IO4)
- net SCL: now also U1.17 (IO22); no longer U1.20 (IO21)
- net SDA: now also U1.20 (IO21); no longer U1.17 (IO22)
- net at D4.2 (A): now also J12.2 (Pin_2); no longer J12.1 (Pin_1)
- net OPTO: now reaches U1.22 (IO18)
- net OPTO: now also R25.1, U3.3
- net GAS1_OUTD: no longer names the net of J4.1 (Pin_1)
- net GAS1_OUTD: now also R21.1, R22.1
- net GAS2_OUTD: no longer names the net of J5.1 (Pin_1)
- net GAS2_OUTD: now also R23.1, R24.1
- new net: J13.1 (Pin_1), U3.1
- new net: J13.2 (Pin_2), U3.2
Other:
- moved on the sheet: J12, J2, J4, J5, R10

Commit message: terminada
Parts:
- removed J8: Placa control, Connector_PinHeader_2.54mm:PinHeader_1x10_P2.54mm_Vertical, symbol Connector:Conn_01x10_Pin
- added J10: Conn_01x06_Pin, Connector_Molex:Molex_KK-254_AE-6410-06A_1x06_P2.54mm_Vertical, symbol Connector:Conn_01x06_Pin
- added J15: Conn_01x04_Pin, Connector_Molex:Molex_KK-254_AE-6410-04A_1x04_P2.54mm_Vertical, symbol Connector:Conn_01x04_Pin
Connections:
- net +3.3V: now also J10.1 (Pin_1)
- net BOTON_1: now also J15.1 (Pin_1)
- net BOTON_2: now also J10.6 (Pin_6)
- net BOTON_3: now also J10.5 (Pin_5)
- net BOTON_4: now also J10.4 (Pin_4)
- net BOTON_5: now also J10.3 (Pin_3)
- net GND: now also J10.2 (Pin_2)
- net LED_1: now also J15.4 (Pin_4)
- net LED_2: now also J15.3 (Pin_3)
- net LED_3: now also J15.2 (Pin_2)
Changed lines of the file:
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@@
 	(wire
 		(pts
-			(xy 76.2 168.91) (xy 80.01 168.91)
+			(xy 76.2 162.56) (xy 80.01 162.56)
 		)
 		(stroke
@@
 	(global_label "BOTON_5"
 		(shape input)
-		(at 76.2 173.99 0)
+		(at 76.2 167.64 0)
 		(fields_autoplaced yes)
 		(effects
@@
 		)
 		(property "Intersheetrefs" "${INTERSHEET_REFS}"
-			(at 87.5914 173.99 0)
+			(at 87.5914 167.64 0)
 			(effects
 				(font
@@
 	(global_label "BOTON_3"
 		(shape input)
-		(at 76.2 179.07 0)
+		(at 76.2 172.72 0)
 		(fields_autoplaced yes)
 		(effects
@@
 		)
 		(property "Intersheetrefs" "${INTERSHEET_REFS}"
-			(at 87.5914 179.07 0)
+			(at 87.5914 172.72 0)
 			(effects
 				(font
@@
 	(global_label "BOTON_2"
 		(shape input)
-		(at 76.2 181.61 0)
+		(at 76.2 175.26 0)
 		(fields_autoplaced yes)
 		(effects
@@
 		)
 		(property "Intersheetrefs" "${INTERSHEET_REFS}"
-			(at 87.5914 181.61 0)
+			(at 87.5914 175.26 0)
 			(effects
 				(font
@@
 	(global_label "BOTON_4"
 		(shape input)
-		(at 76.2 176.53 0)
+		(at 76.2 170.18 0)
 		(fields_autoplaced yes)
 		(effects
@@
 		)
 		(property "Intersheetrefs" "${INTERSHEET_REFS}"
-			(at 87.5914 176.53 0)
+			(at 87.5914 170.18 0)
 			(effects
 				(font
@@
 	(symbol
 		(lib_id "power:+3.3V")
-		(at 80.01 168.91 0)
+		(at 80.01 162.56 0)
 		(unit 1)
 		(exclude_from_sim no)
@@
 		(fields_autoplaced yes)
 		(property "Reference" "#PWR059"
-			(at 80.01 172.72 0)
+			(at 80.01 166.37 0)
 			(effects
 				(font
@@
 		)
 		(property "Value" "+3.3V"
-			(at 80.01 163.83 0)
+			(at 80.01 157.48 0)
 			(effects
 				(font
@@
 		)
 		(property "Footprint" ""
-			(at 80.01 168.91 0)
+			(at 80.01 162.56 0)
 			(effects
 				(font
@@
 		)
 		(property "Datasheet" ""
-			(at 80.01 168.91 0)
+			(at 80.01 162.56 0)
 			(effects
 				(font
@@
 		)
 		(property "Description" "Power symbol creates a global label with name \"+3.3V\""
-			(at 80.01 168.91 0)
+			(at 80.01 162.56 0)
 			(effects
 				(font
@@
 	)
 	(symbol
+		(lib_id "Connector:Conn_01x06_Pin")
+		(at 71.12 167.64 0)
+		(unit 1)
+		(exclude_from_sim no)
+		(in_bom yes)
+		(on_board yes)
+		(dnp no)
+		(fields_autoplaced yes)
+		(property "Reference" "J10"
+			(at 71.755 157.48 0)
+			(effects
+				(font
+					(size 1.27 1.27)
+				)
+			)
+		)
+		(property "Value" "Conn_01x06_Pin"
+			(at 71.755 160.02 0)
+			(effects
+				(font
+					(size 1.27 1.27)
+				)
+			)
+		)
+		(property "Footprint" "Connector_Molex:Molex_KK-254_AE-6410-06A_1x06_P2.54mm_Vertical"
+			(at 71.12 167.64 0)
+			(effects
+				(font
+					(size 1.27 1.27)
+				)
+				(hide yes)
+			)
+		)
+		(property "Datasheet" "~"
+			(at 71.12 167.64 0)
+			(effects
+				(font
+					(size 1.27 1.27)
+				)
+				(hide yes)
+			)
+		)
+		(property "Description" "Generic connector, single row, 01x06, script generated"
+			(at 71.12 167.64 0)
+			(effects
+				(font
+					(size 1.27 1.27)
+				)
+				(hide yes)
+			)
+		)
+		(pin "3"
+		)
+		(pin "6"
+		)
+		(pin "1"
+		)
+		(pin "5"
+		)
+		(pin "2"
+		)
+		(pin "4"
+		)
+		(instances
+			(project ""
+				(path "/65c2dfe9-d457-45cc-a8ad-62a01e187037"
+					(reference "J10")
+					(unit 1)
+				)
+			)
+		)
+	)
+	(symbol
 		(lib_id "Connector:Conn_01x01_Pin")
 		(at 24.13 123.19 0)
@@
 	)
 	(symbol
+		(lib_id "Connector:Conn_01x04_Pin")
+		(at 71.12 186.69 0)
+		(unit 1)
+		(exclude_from_sim no)
+		(in_bom yes)
+		(on_board yes)
+		(dnp no)
+		(property "Reference" "J15"
+			(at 71.12 179.07 0)
+			(effects
+				(font
+					(size 1.27 1.27)
+				)
+			)
+		)
+		(property "Value" "Conn_01x04_Pin"
+			(at 71.12 181.61 0)
+			(effects
+				(font
+					(size 1.27 1.27)
+				)
+			)
+		)
+		(property "Footprint" "Connector_Molex:Molex_KK-254_AE-6410-04A_1x04_P2.54mm_Vertical"
+			(at 71.12 186.69 0)
+			(effects
+				(font
+					(size 1.27 1.27)
+				)
+				(hide yes)
+			)
+		)
+		(property "Datasheet" "~"
+			(at 71.12 186.69 0)
+			(effects
+				(font
+					(size 1.27 1.27)
+				)
+				(hide yes)
+			)
+		)
+		(property "Description" "Generic connector, single row, 01x04, script generated"
+			(at 71.12 186.69 0)
+			(effects
+				(font
+					(size 1.27 1.27)
+				)
+				(hide yes)
+			)
+		)
+		(pin "2"
+		)
+		(pin "3"
+		)
+		(pin "1"
+		)
+		(pin "4"
+		)
+		(instances
+			(project ""
+				(path "/65c2dfe9-d457-45cc-a8ad-62a01e187037"
+					(reference "J15")
+					(unit 1)
+				)
+			)
+		)
+	)
+	(symbol
 		(lib_id "power:GND")
 		(at 36.83 99.06 0)
@@
 	)
 	(symbol
-		(lib_id "Connector:Conn_01x10_Pin")
-		(at 71.12 179.07 0)
-		(unit 1)
-		(exclude_from_sim no)
-		(in_bom yes)
-		(on_board yes)
-		(dnp no)
-		(fields_autoplaced yes)
-		(property "Reference" "J8"
-			(at 71.755 163.83 0)
-			(effects
-				(font
-					(size 1.27 1.27)
-				)
-			)
-		)
-		(property "Value" "Placa control"
-			(at 71.755 166.37 0)
-			(effects
-				(font
-					(size 1.27 1.27)
-				)
-			)
-		)
-		(property "Footprint" "Connector_PinHeader_2.54mm:PinHeader_1x10_P2.54mm_Vertical"
-			(at 71.12 179.07 0)
-			(effects
-				(font
-					(size 1.27 1.27)
-				)
-				(hide yes)
-			)
-		)
-		(property "Datasheet" "~"
-			(at 71.12 179.07 0)
-			(effects
-				(font
-					(size 1.27 1.27)
-				)
-				(hide yes)
-			)
-		)
-		(property "Description" "Generic connector, single row, 01x10, script generated"
-			(at 71.12 179.07 0)
-			(effects
-				(font
-					(size 1.27 1.27)
-				)
-				(hide yes)
-			)
-		)
-		(pin "6"
-		)
-		(pin "5"
-		)
-		(pin "1"
-		)
-		(pin "2"
-		)
-		(pin "7"
-		)
-		(pin "8"
-		)
-		(pin "9"
-		)
-		(pin "10"
-		)
-		(pin "4"
-		)
-		(pin "3"
-		)
-		(instances
-			(project "Placa_perro"
-				(path "/65c2dfe9-d457-45cc-a8ad-62a01e187037"
-					(reference "J8")
-					(unit 1)
-				)
-			)
-		)
-	)
-	(symbol
 		(lib_id "Connector:Conn_01x02_Pin")
 		(at 16.51 24.13 0)
@@
 	(symbol
 		(lib_id "power:GND")
-		(at 76.2 171.45 90)
+		(at 76.2 165.1 90)
 		(unit 1)
 		(exclude_from_sim no)
@@
 		(fields_autoplaced yes)
 		(property "Reference" "#PWR015"
-			(at 82.55 171.45 0)
+			(at 82.55 165.1 0)
 			(effects
 				(font
@@
 		)
 		(property "Value" "GND"
-			(at 80.01 171.4499 90)
+			(at 80.01 165.0999 90)
 			(effects
 				(font
@@
 		)
 		(property "Footprint" ""
-			(at 76.2 171.45 0)
+			(at 76.2 165.1 0)
 			(effects
 				(font
@@
 		)
 		(property "Datasheet" ""
-			(at 76.2 171.45 0)
+			(at 76.2 165.1 0)
 			(effects
 				(font
@@
 		)
 		(property "Description" "Power symbol creates a global label with name \"GND\" , ground"
-			(at 76.2 171.45 0)
+			(at 76.2 165.1 0)
 			(effects
 				(font
