File: Placa_perro/placa_control.kicad_sch (KiCad schematic)
At the start: 17 parts, among them J7 Placa control, SW10 SW_Push, SW11 SW_Push, SW12 SW_Push, SW13 SW_Push, SW9 SW_Push

Commit message: rutee pcb falta molex
Parts:
- added J3: Conn_01x06_Pin, symbol Connector:Conn_01x06_Pin
- added J9: Conn_01x04_Pin, symbol Connector:Conn_01x04_Pin
- D10, D11, D12: footprint LED_THT:LED_D3.0mm_Clear -> LED_THT:LED_D5.0mm
- J7: footprint (none) -> Connector_PinSocket_2.54mm:PinSocket_1x10_P2.54mm_Vertical
Connections:
- net LED_1: now also R17.2; no longer R15.2
- net LED_3: now also R15.2; no longer R17.2
Changed lines of the file:
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@@
 		)
 	)
-	(global_label "LED_3"
+	(global_label "LED_1"
 		(shape input)
 		(at 144.78 60.96 0)
@@
 		)
 	)
-	(global_label "LED_1"
+	(global_label "LED_3"
 		(shape input)
 		(at 146.05 34.29 0)
@@
 			)
 		)
-		(property "Footprint" "LED_THT:LED_D3.0mm_Clear"
+		(property "Footprint" "LED_THT:LED_D5.0mm"
 			(at 133.35 60.96 0)
 			(effects
@@
 			)
 		)
-		(property "Footprint" "LED_THT:LED_D3.0mm_Clear"
+		(property "Footprint" "LED_THT:LED_D5.0mm"
 			(at 134.62 34.29 0)
 			(effects
@@
 			)
 		)
-		(property "Footprint" "LED_THT:LED_D3.0mm_Clear"
+		(property "Footprint" "LED_THT:LED_D5.0mm"
 			(at 134.62 46.99 0)
 			(effects
@@
 	)
 	(symbol
+		(lib_id "Connector:Conn_01x04_Pin")
+		(at 171.45 63.5 0)
+		(unit 1)
+		(exclude_from_sim no)
+		(in_bom yes)
+		(on_board yes)
+		(dnp no)
+		(fields_autoplaced yes)
+		(property "Reference" "J9"
+			(at 172.085 55.88 0)
+			(effects
+				(font
+					(size 1.27 1.27)
+				)
+			)
+		)
+		(property "Value" "Conn_01x04_Pin"
+			(at 172.085 58.42 0)
+			(effects
+				(font
+					(size 1.27 1.27)
+				)
+			)
+		)
+		(property "Footprint" ""
+			(at 171.45 63.5 0)
+			(effects
+				(font
+					(size 1.27 1.27)
+				)
+				(hide yes)
+			)
+		)
+		(property "Datasheet" "~"
+			(at 171.45 63.5 0)
+			(effects
+				(font
+					(size 1.27 1.27)
+				)
+				(hide yes)
+			)
+		)
+		(property "Description" "Generic connector, single row, 01x04, script generated"
+			(at 171.45 63.5 0)
+			(effects
+				(font
+					(size 1.27 1.27)
+				)
+				(hide yes)
+			)
+		)
+		(pin "2"
+		)
+		(pin "3"
+		)
+		(pin "4"
+		)
+		(pin "1"
+		)
+		(instances
+			(project ""
+				(path "/65c2dfe9-d457-45cc-a8ad-62a01e187037/ffefeba4-3dfb-446f-aea2-b2dc01d9727d"
+					(reference "J9")
+					(unit 1)
+				)
+			)
+		)
+	)
+	(symbol
+		(lib_id "Connector:Conn_01x06_Pin")
+		(at 171.45 46.99 0)
+		(unit 1)
+		(exclude_from_sim no)
+		(in_bom yes)
+		(on_board yes)
+		(dnp no)
+		(fields_autoplaced yes)
+		(property "Reference" "J3"
+			(at 172.085 36.83 0)
+			(effects
+				(font
+					(size 1.27 1.27)
+				)
+			)
+		)
+		(property "Value" "Conn_01x06_Pin"
+			(at 172.085 39.37 0)
+			(effects
+				(font
+					(size 1.27 1.27)
+				)
+			)
+		)
+		(property "Footprint" ""
+			(at 171.45 46.99 0)
+			(effects
+				(font
+					(size 1.27 1.27)
+				)
+				(hide yes)
+			)
+		)
+		(property "Datasheet" "~"
+			(at 171.45 46.99 0)
+			(effects
+				(font
+					(size 1.27 1.27)
+				)
+				(hide yes)
+			)
+		)
+		(property "Description" "Generic connector, single row, 01x06, script generated"
+			(at 171.45 46.99 0)
+			(effects
+				(font
+					(size 1.27 1.27)
+				)
+				(hide yes)
+			)
+		)
+		(pin "1"
+		)
+		(pin "6"
+		)
+		(pin "5"
+		)
+		(pin "3"
+		)
+		(pin "4"
+		)
+		(pin "2"
+		)
+		(instances
+			(project ""
+				(path "/65c2dfe9-d457-45cc-a8ad-62a01e187037/ffefeba4-3dfb-446f-aea2-b2dc01d9727d"
+					(reference "J3")
+					(unit 1)
+				)
+			)
+		)
+	)
+	(symbol
 		(lib_id "Connector:Conn_01x10_Pin")
 		(at 191.77 53.34 0)
@@
 			)
 		)
-		(property "Footprint" ""
+		(property "Footprint" "Connector_PinSocket_2.54mm:PinSocket_1x10_P2.54mm_Vertical"
 			(at 191.77 53.34 0)
 			(effects

Commit message: terminada
Parts:
- removed J3: Conn_01x06_Pin, symbol Connector:Conn_01x06_Pin
- removed J7: Placa control, Connector_PinSocket_2.54mm:PinSocket_1x10_P2.54mm_Vertical, symbol Connector:Conn_01x10_Pin
- removed J9: Conn_01x04_Pin, symbol Connector:Conn_01x04_Pin
- added J21: Conn_01x06_Pin, Connector_Molex:Molex_KK-254_AE-6410-06A_1x06_P2.54mm_Vertical, symbol Connector:Conn_01x06_Pin
- added J23: Conn_01x04_Pin, Connector_Molex:Molex_KK-254_AE-6410-04A_1x04_P2.54mm_Vertical, symbol Connector:Conn_01x04_Pin
Connections:
- net +3.3V: now also J21.1 (Pin_1)
- net BOTON_1: now also J23.1 (Pin_1)
- net BOTON_2: now also J21.6 (Pin_6)
- net BOTON_3: now also J21.5 (Pin_5)
- net BOTON_4: now also J21.4 (Pin_4)
- net BOTON_5: now also J21.3 (Pin_3)
- net GND: now also J21.2 (Pin_2)
- net LED_1: now also R16.2, J23.4 (Pin_4); no longer R17.2
- net LED_2: now also R17.2, J23.3 (Pin_3); no longer R16.2
- net LED_3: now also J23.2 (Pin_2)
